File: Electronics/Neopixel - 96 well/Neopixel mini - 96 well.kicad_pcb (KiCad board)
At the start: 2 copper layers, 121.5 x 83 mm, 204 parts, among them J1 Conn_01x03_Male, J2 USB_B, U1 SAMD21_MOD

Commit message: Updated to v1.3
Updated to v1.3. Changes:
- Removed HCC Module footprint from back to simplify design
- Added copper pour to front of PCB for +5V
- Added fiducials for pick and place automation support
Parts:
- removed J2: USB_B, Connectors_USB:USB_Micro-B_Molex-105017-0001
- removed U1: SAMD21_MOD, hcc mod:SAMD_HCC_G_FOOT
- added G***: MapleLogo, logos:MapleLogo, B.Cu at (77.5, 101.0)
Routing:
- net VCC: track 1649.2 -> 1.25 mm, vias 4 -> 0
- net GND: track 1621.3 -> 462.2 mm, vias 0 -> 96
- net Net-(D1-Pad3): track 144.5 -> 41.5 mm, vias 0 -> 2
- net Net-(J2-Pad3): track 15.6 -> 0.00 mm
- net Net-(J2-Pad2): track 15.1 -> 0.00 mm
- net Net-(D48-Pad1): track 110.1 -> 103.6 mm
- net Net-(D60-Pad1): track 105.8 -> 104.4 mm
- net Net-(J2-Pad4): track 0.93 -> 0.00 mm
- added copper zone on F.Cu, net VCC
Other:
- net class 96Mini added: clearance 0.2, trace_width 0.75, via_dia 0.8, via_drill 0.4
- board text added: "4/9/2019"
- board text added: "96 well RGB light guide - v1.3"
- board text added: "DATA"
- board text removed: "3/25/2019"
- board text removed: "96 well RGB light guide - v1.1"
