File: Electronics/Neopixel - 96 well/Neopixel mini - 96 well.sch (KiCad schematic (older format))
At the start: 195 parts, among them J1 Conn_01x03_Male, J2 USB_B, U1 SAMD21_MOD

Commit message: Updated to v1.3
Updated to v1.3. Changes:
- Removed HCC Module footprint from back to simplify design
- Added copper pour to front of PCB for +5V
- Added fiducials for pick and place automation support
Parts:
- removed J2: USB_B, Connectors_USB:USB_Micro-B_Molex-105017-0001, symbol Connector:USB_B
- removed U1: SAMD21_MOD, hcc mod:SAMD_HCC_G_FOOT, symbol samd_hcc_mod:SAMD21_MOD
Connections:
- wire segments 939 -> 909
Changed lines of the file:
@@
 $EndComp
 Wire Wire Line
-	7500 1925 7150 1925
-Wire Wire Line
-	7150 1925 7150 2500
-Connection ~ 7500 1925
-Wire Wire Line
 	7550 3575 7150 3575
 Wire Wire Line
-	7150 3575 7150 3200
-Wire Wire Line
-	7275 2050 7275 2775
-Wire Wire Line
 	7275 2825 7150 2825
 $Comp
@@
 Wire Wire Line
 	8475 1975 8475 2350
-$Comp
-L samd_hcc_mod:SAMD21_MOD U1
-U 1 1 5D91C257
-P 4350 4450
-F 0 "U1" H 4725 6397 60  0000 C CNN
-F 1 "SAMD21_MOD" H 4725 6291 60  0000 C CNN
-F 2 "hcc mod:SAMD_HCC_G_FOOT" H 4350 4450 60  0001 C CNN
-F 3 "" H 4350 4450 60  0001 C CNN
-	1    4350 4450
-	1    0    0    -1
-$EndComp
-Wire Wire Line
-	6400 3150 5650 3150
-Wire Wire Line
-	5650 3250 5650 3150
-Connection ~ 5650 3150
-Wire Wire Line
-	6400 2925 6400 3150
-Wire Wire Line
-	6125 2825 6125 3900
-Wire Wire Line
-	6125 3900 4900 3900
-$Comp
-L Connector:USB_B J2
-U 1 1 5DCB9033
-P 3350 2350
-F 0 "J2" H 3405 2817 50  0000 C CNN
-F 1 "USB_B" H 3405 2726 50  0000 C CNN
-F 2 "Connectors_USB:USB_Micro-B_Molex-105017-0001" H 3500 2300 50  0001 C CNN
-F 3 " ~" H 3500 2300 50  0001 C CNN
-	1    3350 2350
-	1    0    0    -1
-$EndComp
-Wire Wire Line
-	3650 2150 5750 2150
-Wire Wire Line
-	5750 2150 5750 2850
-Wire Wire Line
-	5750 2850 5700 2850
-Wire Wire Line
-	3650 2350 5875 2350
-Wire Wire Line
-	5875 2350 5875 3050
-Wire Wire Line
-	5875 3050 5650 3050
-Wire Wire Line
-	3650 2450 5725 2450
-Wire Wire Line
-	5725 2450 5725 2950
-Wire Wire Line
-	5725 2950 5650 2950
-Wire Wire Line
-	5700 2725 5700 2850
-Connection ~ 5700 2850
-Wire Wire Line
-	5700 2850 5650 2850
-Wire Wire Line
-	6400 2925 6700 2925
-Wire Wire Line
-	6700 2925 6700 3200
-Wire Wire Line
-	6700 3200 7150 3200
-Connection ~ 7150 3200
-Wire Wire Line
-	7150 3200 7150 2925
-Wire Wire Line
-	6850 2825 6850 2775
-Wire Wire Line
-	6850 2775 7275 2775
-Wire Wire Line
-	6850 2825 6125 2825
-Connection ~ 7275 2775
-Wire Wire Line
-	7275 2775 7275 2825
-Wire Wire Line
-	6850 2725 6850 2500
-Wire Wire Line
-	6850 2500 7150 2500
+Connection ~ 7500 1925
 Wire Wire Line
-	6850 2725 5700 2725
-Connection ~ 7150 2500
+	7500 1925 7150 1925
 Wire Wire Line
-	7150 2500 7150 2725
+	7150 1925 7150 2725
 Wire Wire Line
-	3250 2750 3250 3250
+	7150 2925 7150 3575
 Wire Wire Line
-	3250 3250 5650 3250
+	7275 2050 7275 2825
 $EndSCHEMATC
